File: festBin_eagle/festBin.brd (EAGLE design)
At the start: 144.8 x 135.6 mm, 47 parts, among them IC1 74LS14N, K1 4052, K2 4052, Q1 BD139, Q2 BD139

Commit message: ver_0.6_clean
Parts:
- removed C10: 10u, rcl:E2,5-6
- removed R16: 1k, rcl:0207/10
- removed R17: 47k, rcl:0207/10
- removed R18: 10k, rcl:0207/10
- added C3: 10u, rcl:E2,5-6
- added R11, R12: 1k, rcl:0207/10
- added R7: 10k, rcl:0207/10
- C5: value 100n -> 0.33u
- C6: value 0.33u -> 100n
- OK2: value PC817 -> 4N33; device optocoupler:DIL04 -> optocoupler:DIL06
- OK3: value 4N33 -> PC817; device optocoupler:DIL06 -> optocoupler:DIL04
- R1: value 2.2k -> 10k
- R4: value 1k -> 47k
- R5: value 10k -> 2k
- R6: value 2k -> 2.2k
- moved R6 86.0 mm to (46.6, 68.0), turned to 180 degrees
- moved R4 83.6 mm to (40.2, 45.7)
- moved R3 79.3 mm to (65.7, 79.9)
- moved R5 73.6 mm to (132.1, 77.5), turned to 270 degrees
- moved K1 50.0 mm to (26.4, 27.5), turned to 90 degrees
- moved K2 50.0 mm to (26.7, 77.5), turned to 270 degrees
- moved C1 37.7 mm to (57.8, 26.7), turned to 180 degrees
- moved R1 33.2 mm to (65.8, 40.9), turned to 0 degrees
- moved OK3 21.8 mm to (47.1, 86.8), turned to 90 degrees
- moved R2 20.2 mm to (66.0, 45.0), turned to 0 degrees
- moved OK2 13.8 mm to (60.0, 69.2), turned to 270 degrees
- moved OK1 11.3 mm to (47.7, 75.5)
- moved Q1 11.2 mm to (37.3, 74.8)
- moved Q2 11.2 mm to (36.6, 86.0)
- moved LED1 5.48 mm to (56.2, 79.9)
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- renumbered C11 to C6, C12 to C5, C9 to C4, D6 to D2, D7 to D1, IC4 to IC2, R14 to R9, R15 to R10, R19 to R8
Connections:
- removed net N$11 (its old number): OK2.3, Q2.B
- removed net N$18 (its old number): LED2.K, OK2.1
- new net N$19: LED2.K, OK3.1
- new net N$24: OK3.3, Q2.B
- net +5V: now also R1.2, R7.2; no longer R18.2, R5.2
- net C_L_I: now also R11.1; no longer R3.1
- net D_L_I: now also R12.1; no longer R4.1
- net GND: now also C3.-, OK2.4, R5.1; no longer C10.-, OK3.4, R6.1
- net MOT_B: now also K1.P1, K1.P2; no longer K2.P1, K2.P2
- net MOT_F: now also K2.P1, K2.P2; no longer K1.P1, K1.P2
- net M_B: now also R3.2; no longer R16.2
- net N$1: now also R6.2; no longer R1.2
- net N$10: now also OK3.4; no longer OK1.4
- net N$12: now also K2.2, Q2.C; no longer K1.2, Q1.C
- net N$2: now also C1.+, R1.1; no longer C10.+, R18.1
- net N$21: now also OK1.4, R4.2; no longer OK2.4, R17.2
- net N$23: now also K1.2, Q1.C; no longer K2.2, Q2.C
- net N$25: now also OK2.1, R6.1; no longer OK3.1, R1.1
- net N$26: now also C3.+, OK2.5, R7.1; no longer C1.+, OK3.5, R2.1
- net N$3: now also R11.2; no longer R3.2
- net N$4: now also R12.2; no longer R4.2
- net N$5: now also R2.1; no longer R5.1
- net N$6: now also LED2.A; no longer LED1.A
- net N$7: now also LED1.A, R3.1; no longer LED2.A, R16.1
- net VCC: now also R4.1; no longer R17.1
- net W_S: now also R5.2; no longer R6.2
Routing:
- net N$18 (its old number): track 8.45 -> 0.00 mm
- net N$24: track 0.00 -> 5.46 mm
- net N$11 (its old number): track 5.43 -> 0.00 mm
- net N$18: track 4.14 -> 8.45 mm
- net N$19: track 0.00 -> 4.14 mm
