File: festBin_eagle/festBin.sch (EAGLE design)
At the start: 47 parts, among them IC1 74LS14N, K1 4052, K2 4052, Q1 BD139, Q2 BD139

Commit message: ver_0.6_clean
Parts:
- removed C10: 10u, rcl:CPOL-EUE2.5-6
- removed R16: 1k, rcl:R-EU_0207/10
- removed R17: 47k, rcl:R-EU_0207/10
- removed R18: 10k, rcl:R-EU_0207/10
- added C3: 10u, rcl:CPOL-EUE2.5-6
- added R11, R12: 1k, rcl:R-EU_0207/10
- added R7: 10k, rcl:R-EU_0207/10
- C5: value 100n -> 0.33u
- C6: value 0.33u -> 100n
- OK2: value PC817 -> 4N33; device optocoupler:PC817 -> optocoupler:4N33
- OK3: value 4N33 -> PC817; device optocoupler:4N33 -> optocoupler:PC817
- R1: value 2.2k -> 10k
- R4: value 1k -> 47k
- R5: value 10k -> 2k
- R6: value 2k -> 2.2k
- renumbered C11 to C6, C12 to C5, C9 to C4, D6 to D2, D7 to D1, IC4 to IC2, R14 to R9, R15 to R10, R19 to R8
Connections:
- removed net N$11 (its old number): OK2.EMIT, Q2.B
- removed net N$18 (its old number): LED2.C, OK2.A
- new net N$19: LED2.C, OK3.A
- new net N$24: OK3.EMIT, Q2.B
- net +5V: now also R1.2, R7.2; no longer R18.2, R5.2
- net C_L_I: now also R11.1; no longer R3.1
- net D_L_I: now also R12.1; no longer R4.1
- net GND: now also C3.-, OK2.E, R5.1; no longer C10.-, OK3.E, R6.1
- net MOT_B: now also K12.P, K13.P; no longer K22.P, K23.P
- net MOT_F: now also K22.P, K23.P; no longer K12.P, K13.P
- net M_B: now also R3.2; no longer R16.2
- net N$1: now also R6.2; no longer R1.2
- net N$10: now also OK3.COL; no longer OK1.COL
- net N$12: now also K21.2, Q2.C; no longer K11.2, Q1.C
- net N$2: now also C1.+, R1.1; no longer C10.+, R18.1
- net N$21: now also OK1.COL, R4.2; no longer OK2.COL, R17.2
- net N$23: now also K11.2, Q1.C; no longer K21.2, Q2.C
- net N$25: now also OK2.A, R6.1; no longer OK3.A, R1.1
- net N$26: now also C3.+, OK2.COL, R7.1; no longer C1.+, OK3.COL, R2.1
- net N$3: now also R11.2; no longer R3.2
- net N$4: now also R12.2; no longer R4.2
- net N$5: now also R2.1; no longer R5.1
- net N$6: now also LED2.A; no longer LED1.A
- net N$7: now also LED1.A, R3.1; no longer LED2.A, R16.1
- net VCC: now also R4.1; no longer R17.1
- net W_S: now also R5.2; no longer R6.2
Other:
- moved on the sheet: C1, K1, K2, LED1, LED2, OK1, Q1, Q2, R1, R2, R3, R4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
